Commit message: fix

File: solidworks/swerve_urdf/urdf/swerve_urdf.urdf (robot description, URDF)
Before this commit: robot swerve_urdf, 9 links, 8 joints
Links:
- link drive2: mass 0.093012494318941 -> 0.0930124943189411
Joints:
- joint drive1_joint: origin xyz=0 0.016 -0.04757 rpy=1.5708 0 3.1416 -> xyz=0 0.0159999999998657 -0.0475700189392033 rpy=1.5707963267949 0 3.14159265358979
- joint drive3_joint: axis 0 1 0 -> 0 0 1; origin xyz=0 0 0 rpy=0 0 0 -> xyz=0 0.016 -0.04757 rpy=1.5708 0 3.1416
- joint steer1_joint: origin xyz=0.178 -0.178 0.01157 rpy=0 0 0 -> xyz=0.177999999999973 -0.177999999999867 0.0115700189392032 rpy=0 0 0
- joint steer2_joint: origin xyz=0.178 0.178 0.01157 rpy=0 0 0 -> xyz=0.177999999999971 0.178000000000137 0.0115700189392031 rpy=0 0 0
